Commit message: add rune record

File: rm_vision/rm_gimbal_description/urdf/rm_gimbal.urdf.xacro (robot description, xacro)
@@ -1,6 +1,6 @@
 <?xml version="1.0" encoding="utf-8"?>
 <robot name="rm_gimbal" xmlns:xacro="http://ros.org/wiki/xacro">
-  <xacro:arg name="odom2gimbal" default="-0.190 0.017 0.043" />
-  <xacro:arg name="giambal2camera" default="0.152 -0.017 0.0 " />
+  <xacro:arg name="odom2gimbal" default="0.0828 0.013 -0.0434" />
+  <xacro:arg name="giambal2camera" default="0.0838 0.0 0.0437 " />
   <!-- <xacro:arg name="giambal2camera" default="0.1 -0.06 0.00 " /> -->
   <xacro:arg name="rpy" default="0 0 0" />
@@ -20,6 +20,7 @@
   <link name="camera_link" />
   <joint name="camera_optical_joint" type="fixed">
-    <origin xyz="0 0 0" rpy="-1.579522 0 ${-pi/2}" />
-    <!-- <origin xyz="0 0 0" rpy="${-pi/2} 0 ${-pi/2}" /> -->
+    <!-- <origin xyz="0 0 0" rpy="-1.579522 0 ${-pi/2}" /> -->
+    <origin xyz="0 0 0" rpy="${-pi/2} 0 ${-pi/2}" />
+    <!-- <origin xyz="0 0 0" rpy="-1.560478 0 ${-pi/2}" /> -->
     <parent link="camera_link" />
     <child link="camera_optical_frame" />
